File: KiCAD_Files/FreeDSP_INTEGRA_PANELBOARD/FreeDSP_INTEGRA_PANELBOARD.kicad_sch (KiCad schematic)
At the start: 50 parts, among them J1 Conn_01x04, J2 Header_01x06, J3 Conn_01x08, SW1 EN11-HSB1AF15, SW2 SW_PUSH, U1 OSRB38C9AA, U2 OSL40391-IX, U3 PIC16F1938-I/SP

Commit message: Add files via upload
Fix some values.
Parts:
- C1: JLPCB# C14663 -> HAND
- C2, C3: JLPCB# C28233 -> HAND
- C4: JLPCB# C45783 -> NOP; now not fitted
- D1, D2, D6, D7, D9: JLPCB# C81598 -> HAND
- D3, D4, D5, D8, R2, R3: JLPCB# (none) -> HAND
- J1: now not fitted
- MH3: now left out of the parts list
- R1, R8: value 430R -> 1k; JLPCB# (none) -> HAND
- R10, R11, R12, R13, R14, R15, R16, R9: JLPCB# C4275 -> HAND
- R17, R18: JLPCB# C21189 -> HAND
- R19, R20, R21, R5, R6, R7: JLPCB# C25804 -> HAND
- R22, R23, R24, R25: JLPCB# C23140 -> HAND
- R4: JLPCB# C31850 -> HAND
Other:
- note added: "（ANODE COMMON)"
- moved on the sheet: D9, J2, R20

Commit message: Parts value changed
Parts:
- C2: now fitted
- D3, D4, D5, D8: value LED_RED -> LED_YELLOW
- R10, R11, R12, R13, R14, R15, R16, R9: value 75R -> 47R
- R2, R3: value 390R -> 470R
- R22, R23, R24, R25: value 33R -> 47R
Changed lines of the file:
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@@
 		(title "TAS6422 FreeDSP INTEGRA Remote")
 		(date "2026-03-31")
-		(rev "0.11")
+		(rev "0.12")
 		(company "Designed by CyberPit HILO 2026")
 		(comment 4 "User Interfaces, TAS6424 Power Amplifier Part, Root Schematic")
@@
 			)
 		)
-		(property "Value" "33R"
+		(property "Value" "47R"
 			(at 210.185 104.14 90)
 			(effects
@@
 			)
 		)
-		(property "Value" "75R"
+		(property "Value" "47R"
 			(at 167.64 135.89 90)
 			(effects
@@
 			)
 		)
-		(property "Value" "LED_RED"
+		(property "Value" "LED_YELLOW"
 			(at 143.51 42.2401 90)
 			(effects
@@
 			)
 		)
-		(property "Value" "390R"
+		(property "Value" "470R"
 			(at 77.47 33.02 90)
 			(effects
@@
 			)
 		)
-		(property "Value" "75R"
+		(property "Value" "47R"
 			(at 167.64 133.35 90)
 			(effects
@@
 			)
 		)
-		(property "Value" "75R"
+		(property "Value" "47R"
 			(at 167.64 128.27 90)
 			(effects
@@
 					(size 1.27 1.27)
 				)
+				(hide yes)
 			)
 		)
@@
 			)
 		)
-		(property "Value" "LED_RED"
+		(property "Value" "LED_YELLOW"
 			(at 54.61 34.6201 90)
 			(effects
@@
 			)
 		)
-		(property "Value" "75R"
+		(property "Value" "47R"
 			(at 167.64 143.51 90)
 			(effects
@@
 			)
 		)
-		(property "Value" "75R"
+		(property "Value" "47R"
 			(at 167.64 138.43 90)
 			(effects
@@
 			)
 		)
-		(property "Value" "LED_RED"
+		(property "Value" "LED_YELLOW"
 			(at 81.28 42.2401 90)
 			(effects
@@
 			)
 		)
-		(property "Value" "75R"
+		(property "Value" "47R"
 			(at 167.64 125.73 90)
 			(effects
@@
 			)
 		)
-		(property "Value" "LED_RED"
+		(property "Value" "LED_YELLOW"
 			(at 109.22 43.5101 90)
 			(effects
@@
 			)
 		)
-		(property "Value" "33R"
+		(property "Value" "47R"
 			(at 210.185 106.68 90)
 			(effects
@@
 			)
 		)
-		(property "Value" "75R"
+		(property "Value" "47R"
 			(at 167.64 130.81 90)
 			(effects
@@
 			)
 		)
-		(property "Value" "75R"
+		(property "Value" "47R"
 			(at 167.64 140.97 90)
 			(effects
@@
 		(in_bom yes)
 		(on_board yes)
-		(dnp yes)
+		(dnp no)
 		(property "Reference" "C2"
 			(at 147.955 179.07 90)
@@
 			)
 		)
-		(property "Value" "390R"
+		(property "Value" "470R"
 			(at 105.41 34.29 90)
 			(effects
@@
 			)
 		)
-		(property "Value" "33R"
+		(property "Value" "47R"
 			(at 210.185 109.22 90)
 			(effects
@@
 			)
 		)
-		(property "Value" "33R"
+		(property "Value" "47R"
 			(at 210.185 111.76 90)
 			(effects
