File: KiCAD_Files/FreeDSP_INTEGRA_QUAD-PRO/Audio_ADC.kicad_sch (KiCad schematic)
At the start: 119 parts, among them IC3 AK5574EN, IC4 OPA1632DR, IC5 OPA1632DR, J13 MJ518A/RCJ2123, J14 Molex_MPJ-8004-3P, J15 Molex_MPJ-8004-3P, J16 Conn_01x02, J17 PinHeader_02x02, Q13 2N7002, U15 OPA1612AIDR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

Commit message: Add files via upload
Parts:
- C131, C132, C136, C137: value 10uF/16V -> 22uF/16V
Other:
- note added: "24.576MHz (32x8fs)"
- note added: "96kHz(fs)"
- note added: "ADC = MASTER fs = 96kHz Format = 8Slots TDM LEFT = (ADC1-ADC2)/2 RIGHT = (ADC3-ADC4)/2"
- note removed: "3072kHz"
- note removed: "ADC = MASTER fs = 96kHz Format = I4S or TDM LEFT = (ADC1-ADC2)/2 RIGHT = (ADC3-ADC4)/2"
- note removed: "fs=48kHz I2S"
- moved on the sheet: C131, C132, C136, C137
