File: KiCAD_Files/FreeDSP_INTEGRA_QUAD-PRO/Micom_Display.kicad_sch (KiCad schematic)
At the start: 41 parts, among them J18 Conn_01x04, J19 OSRB38C9AA, J20 Header_01x06, J21 Conn_01x04, J22 Conn_01x08, SW6 SW_PUSH, SW7 EN11-HSB1AF15, U17 OSL40391-IX, U18 PIC16F1938-I/SP

Commit message: Add files via upload
Changed lines of the file:
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@@
 		(title "TAS6422 FreeDSP INTEGRA QUAD PRO")
 		(date "2026-02-07")
-		(rev "0.4")
+		(rev "0.41")
 		(company "Designed by CyberPit HILO 2026")
 		(comment 4 "Micom Contriller Display interface part")
@@
 	(polyline
 		(pts
-			(xy 102.87 104.14) (xy 103.505 104.14)
+			(xy 102.87 103.124) (xy 103.505 103.124)
 		)
 		(stroke
@@
 	(polyline
 		(pts
-			(xy 102.87 99.06) (xy 102.87 104.14)
+			(xy 102.87 98.806) (xy 102.87 103.124)
 		)
 		(stroke
@@
 	(polyline
 		(pts
-			(xy 100.965 101.6) (xy 100.965 82.55)
+			(xy 100.838 101.092) (xy 100.838 82.55)
 		)
 		(stroke
@@
 	(polyline
 		(pts
+			(xy 97.79 104.394) (xy 97.79 71.12)
+		)
+		(stroke
+			(width 0)
+			(type default)
+		)
+	)
+	(polyline
+		(pts
 			(xy 138.43 118.11) (xy 136.525 118.745)
 		)
@@
 	(polyline
 		(pts
-			(xy 100.965 82.55) (xy 101.6 81.915)
+			(xy 100.838 82.55) (xy 101.6 81.915)
 		)
 		(stroke
@@
 		)
 	)
+	(polyline
+		(pts
+			(xy 97.79 71.12) (xy 98.552 70.358)
+		)
+		(stroke
+			(width 0)
+			(type default)
+		)
+	)
 	(wire
 		(pts
@@
 		)
 	)
+	(polyline
+		(pts
+			(xy 98.552 70.358) (xy 104.648 70.358)
+		)
+		(stroke
+			(width 0)
+			(type default)
+		)
+	)
 	(wire
 		(pts
@@
 	(polyline
 		(pts
-			(xy 102.87 99.06) (xy 103.505 99.06)
+			(xy 102.87 98.806) (xy 103.378 98.806)
 		)
 		(stroke
@@
 		)
 	)
+	(polyline
+		(pts
+			(xy 97.79 104.394) (xy 103.632 104.394)
+		)
+		(stroke
+			(width 0)
+			(type default)
+		)
+	)
 	(wire
 		(pts
@@
 	(polyline
 		(pts
-			(xy 100.965 101.6) (xy 102.87 101.6)
+			(xy 100.838 101.092) (xy 102.87 101.092)
 		)
 		(stroke
@@
 				(margins 0.9525 0.9525 0.9525 0.9525)
 				(span 1 1)
+				(fill
+					(type none)
+				)
+				(effects
+					(font
+						(size 1.27 1.27)
+					)
+					(justify left top)
+				)
+			)
+		)
+	)
+	(table
+		(column_count 2)
+		(border
+			(external yes)
+			(header yes)
+			(stroke
+				(width 0.508)
+				(type solid)
+			)
+		)
+		(separators
+			(rows yes)
+			(cols yes)
+			(stroke
+				(width 0)
+				(type solid)
+			)
+		)
+		(column_widths 9.525 21.59)
+		(row_heights 3.81 2.54 2.54)
+		(cells
+			(table_cell "bit2"
+				(exclude_from_sim no)
+				(at 104.775 68.58 0)
+				(size 9.525 3.81)
+				(margins 0.9525 0.9525 0.9525 0.9525)
+				(span 1 1)
+				(fill
+					(type color)
+					(color 161 255 249 1)
+				)
+				(effects
+					(font
+						(size 1.27 1.27)
+					)
+				)
+			)
+			(table_cell "BTL MODE"
+				(exclude_from_sim no)
+				(at 114.3 68.58 0)
+				(size 21.59 3.81)
+				(margins 0.9525 0.9525 0.9525 0.9525)
+				(span 1 1)
+				(fill
+					(type color)
+					(color 161 255 249 1)
+				)
+				(effects
+					(font
+						(size 1.27 1.27)
+					)
+				)
+			)
+			(table_cell "H"
+				(exclude_from_sim no)
+				(at 104.775 72.39 0)
+				(size 9.525 2.54)
+				(margins 0.9525 0.9525 0.9525 0.9525)
+				(span 1 1)
+				(fill
+					(type none)
+				)
+				(effects
+					(font
+						(size 1.27 1.27)
+					)
+				)
+			)
+			(table_cell "PBTL (2ch)"
+				(exclude_from_sim no)
+				(at 114.3 72.39 0)
+				(size 21.59 2.54)
+				(margins 0.9525 0.9525 0.9525 0.9525)
+				(span 1 1)
+				(fill
+					(type none)
+				)
+				(effects
+					(font
+						(size 1.27 1.27)
+					)
+					(justify left top)
+				)
+			)
+			(table_cell "L"
+				(exclude_from_sim no)
+				(at 104.775 74.93 0)
+				(size 9.525 2.54)
+				(margins 0.9525 0.9525 0.9525 0.9525)
+				(span 1 1)
+				(fill
+					(type none)
+				)
+				(effects
+					(font
+						(size 1.27 1.27)
+					)
+				)
+			)
+			(table_cell "BTL (4ch)"
+				(exclude_from_sim no)
+				(at 114.3 74.93 0)
+				(size 21.59 2.54)
+				(margins 0.9525 0.9525 0.9525 0.9525)
+				(span 1 1)
