File: KiCAD_Files/FreeDSP_INTEGRA_QUAD-PRO/YAM_DSP-ADC_IO.kicad_sch (KiCad schematic)
At the start: 166 parts, among them J10 Conn_01x05, J11 Header_01x04, J12 Header_01x06, J6 Conn_Coaxial, J8 Conn_01x02, J9 IDC_2x5, P1 Conn_02x20_Odd_Even, Q11 AO3400A, Q12 2N7002, Q5 2N7002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

Commit message: Add files via upload
Parts:
- J10: value Conn_01x05 -> Header_01x06
Changed lines of the file:
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@@
 		(title "TAS6422 FreeDSP INTEGRA QUAD PRO")
 		(date "2026-03-15")
-		(rev "0.4")
+		(rev "0.41")
 		(company "Designed by CyberPit HILO 2026")
 		(comment 4 "DSP, Wireless, S/PDIF interface part")
@@
 			)
 		)
-		(property "Value" "Conn_01x05"
+		(property "Value" "Header_01x06"
 			(at 213.36 88.9 0)
 			(effects
