File: KiCAD_Files/FreeDSP_INTEGRA_QUAD-PRO/YAM_PSU_IO.kicad_sch (KiCad schematic)
At the start: 114 parts, among them J3 Barrel_Jack_2DC-G213-D42, J4 Screw_Terminal_01x02, J5 Screw_Terminal_01x02, Q2 MMBT5401, Q3 MMBT5401, Q4 2N7002, U19 TPS5430DDAR, U2 TPS5430DDAR, U3 LM2611AMFX, U4 LM317AG-TN3-R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

Commit message: Add files via upload
Parts:
- C31: value 22uF/16V -> 22uF/25V
- C39, C41, C43, C44, C45, C47, C50, C52: value 470uF/25V_OS -> 820uF/25V_OS
Changed lines of the file:
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@@
 	(title_block
 		(title "TAS6422 FreeDSP INTEGRA QUAD PRO")
-		(date "2026-02-07")
-		(rev "0.4")
+		(date "2026-05-19")
+		(rev "0.41")
 		(company "Designed by CyberPit HILO 2026")
 		(comment 4 "Power Supply Unit part")
@@
 			)
 		)
-		(property "Value" "22uF/16V"
+		(property "Value" "22uF/25V"
 			(at 80.01 165.1 90)
 			(effects
 				(font
 					(size 1.27 1.27)
+					(thickness 0.254)
+					(bold yes)
 				)
 			)
@@
 		)
 		(property "Value" "0.1uF/50V"
-			(at 81.28 230.505 90)
+			(at 81.026 229.87 90)
 			(effects
 				(font
@@
 			)
 		)
-		(property "Value" "470uF/25V_OS"
+		(property "Value" "820uF/25V_OS"
 			(at 120.65 242.57 90)
 			(effects
@@
 			)
 		)
-		(property "Value" "470uF/25V_OS"
+		(property "Value" "820uF/25V_OS"
 			(at 127 242.57 90)
 			(effects
@@
 			)
 		)
-		(property "Value" "470uF/25V_OS"
+		(property "Value" "820uF/25V_OS"
 			(at 133.35 242.57 90)
 			(effects
@@
 			)
 		)
-		(property "Value" "470uF/25V_OS"
+		(property "Value" "820uF/25V_OS"
 			(at 139.7 242.57 90)
 			(effects
@@
 			)
 		)
-		(property "Value" "470uF/25V_OS"
+		(property "Value" "820uF/25V_OS"
 			(at 146.05 242.57 90)
 			(effects
@@
 			)
 		)
-		(property "Value" "470uF/25V_OS"
+		(property "Value" "820uF/25V_OS"
 			(at 152.4 242.57 90)
 			(effects
@@
 			)
 		)
-		(property "Value" "470uF/25V_OS"
+		(property "Value" "820uF/25V_OS"
 			(at 158.75 242.57 90)
 			(effects
@@
 			)
 		)
-		(property "Value" "470uF/25V_OS"
+		(property "Value" "820uF/25V_OS"
 			(at 165.1 242.57 90)
 			(effects
